File: FT230X-Serial-Board/FT230X-Serial-Board.kicad_pcb (KiCad board)
At the start: 4 copper layers, 34 x 19.3 mm, 31 parts, among them J1 USB_C_Receptacle_USB2.0, J2 Conn_01x08_Male, J3 Conn_01x08_Male, J4 Conn_01x04_Male, U1 FT230XQ

Commit message: Fixed errors on FT230X-Serial-Board.
Parts:
- R10, R9: value 270 -> 4k7
Changed lines of the file:
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@@
     (add_net /VUSB_SENSE)
     (add_net GND)
+    (add_net "Net-(J1-PadA8)")
+    (add_net "Net-(J1-PadB8)")
     (add_net "Net-(LED1-Pad1)")
     (add_net "Net-(LED2-Pad1)")
@@
       (effects (font (size 0.8 0.8) (thickness 0.15)))
     )
-    (fp_text value 270 (at 0 1.17) (layer F.Fab)
+    (fp_text value 4k7 (at 0 1.17) (layer F.Fab)
       (effects (font (size 1 1) (thickness 0.15)))
     )
@@
       (effects (font (size 0.8 0.8) (thickness 0.15)))
     )
-    (fp_text value 270 (at 0 1.17) (layer F.Fab)
+    (fp_text value 4k7 (at 0 1.17) (layer F.Fab)
       (effects (font (size 1 1) (thickness 0.15)))
     )
