File: ESP8266-Cherry-MX-Board/ESP8266-Cherry-MX-Board.kicad_pcb (KiCad board)
At the start: 2 copper layers, 33 x 90 mm, 63 parts, among them J1 Conn_01x04_Male, J2 USB_C_Receptacle_USB2.0, J3 Conn_01x02, J4 Conn_01x07_Male, SW1 SW_SPST, SW2 SW_SPST, SW3 SW_SPST, SW4 SW_SPST, SW5 PEC11L-4115F-S0020, SW7 SW_Push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

Commit message: Fixed errors on ESP8266-Cherry-MX-Board.
Parts:
- added R27: 10k, Resistor_SMD:R_0603_1608Metric, F.Cu at (162.0, 52.0)
- added R28: 10k, Resistor_SMD:R_0603_1608Metric, F.Cu at (162.0, 53.5)
- R25: value 100k -> 499k
- R26: value 499k -> 100k
Routing:
- net +3V3: track 277.1 -> 279.3 mm
- net /GPIO15: track 46.8 -> 47.6 mm
- net /GPIO2: track 46.3 -> 47.0 mm

Commit message: Updated component values.
Parts:
- R15, R18: value 10k -> 0R
